File: CoffeeMakersch.sch (EAGLE design)
At the start: 25 parts, among them K1 G5LE

Commit message: Finished schematic
Parts:
- added C13, C14, C15, C16, C18, C22, C23, C24: 100n, rcl:C-USC0805
- added C17: 10u, rcl:C-USC0805
- added C19, C20, C21: 10n, rcl:C-USC0805
- added C25: 4.7u, rcl:C-USC0805
- added C26, C27, C28, C29, C30: 470u, rcl:CPOL-USUD-10X10
- added D1: BAS70, diode:BAS70
- added LED1: (no value), led:LEDCHIPLED_1206
- added R10, R11, R12, R13, R4, R8, R9: 10k, rcl:R-US_R0805
- added R2: 330, rcl:R-US_R0805
- added R3: 27k, rcl:R-US_R0805
- added R7: 1M, rcl:R-US_R0805
- added S1, S2: (no value), switch-omron:10-XX
- added U$10, U$9: 5TERM, EmbSystems:5TERM
- added U$11: ADAFRUIT_128X32, EmbSystems:ADAFRUIT_128X32
- added U$12: 5TERM-3, EmbSystems:5TERM-3
- added U$13: LD117-5, EmbSystems:LD117-5
- added U$14: 74LVC, EmbSystems:74LVC
- added U$15: LMV321LICT, EmbSystems:LMV321LICT
- added U$16: NC7SZ04, EmbSystems:NC7SZ04
- C1, C10, C8: value (none) -> 4.7u
- C11: value (none) -> 1u
- C12: value (none) -> 10n
- C2, C3, C4, C5, C6, C7, C9: value (none) -> 100n
Connections:
- new net 5V: C30.+, R2.2, U$12.P$3, U$13.VOUT, U$14.VCCB
- new net ADC_IN1: U$1.PA1, U$2.OUT, U$2.SENSE
- new net BREW: S2.S, S2.S1, U$1.PA6
- new net DAC_OUT1: U$1.PA4, U$7.+IN
- new net ENCA: C20.1, R10.2, U$1.PA2
- new net ENCB: C21.1, R11.1, U$1.PA3
- new net FLOW: U$1.PA5, U$14.A
- new net I2C1_SCL: U$1.PB6, U$11.SCL
- new net I2C1_SDA: U$1.PB7, U$11.SDA
- new net N$10: C19.2, U$7.COMP
- new net N$11: C19.1, D1.C, R3.2, U$10.P$1, U$7.OUT
- new net N$12: R3.1, R4.2, U$7.-IN
- new net N$13: R10.1, R12.2, U$4.A
- new net N$14: R11.2, R13.2, U$4.B, U$4.B@2
- new net N$15: U$15.IN-, U$15.OUT, U$7.S/D
- new net N$17: U$12.P$1, U$14.B
- new net N$5: LED1.A, R2.1
- new net N$6: C13.1, R7.1, R9.2, U$2.-IN
- new net N$7: C14.1, R8.1, U$2.+IN
- new net N$8: C15.1, R8.2, U$9.P$2
- new net N$9: C15.2, R9.1, U$9.P$1
- new net NRST: U$1.NRST, U$16.OUT
- new net PA10: SV2.2, U$1.PA10
- new net PA9: SV2.1, U$1.PA9
- new net PC4: SV1.2, U$1.PC4
- new net PC5: SV1.1, U$1.PC5
- new net PUMPSHUTDOWN: U$1.PB15, U$15.IN+
- new net RELAY: K11.1, U$1.PB12
- new net RST: S1.S, S1.S1
- new net SRST: U$1.PB5, U$11.RST
- new net SW: U$1.PA0, U$4.SW
- net 12V: now also C26.+, C27.+, C28.+, U$13.VIN, U$3.+VDC, U$7.V+
- net 3V3: now also C11.1, C12.1, C16.1, C17.1, C22.1, C23.1, C24.1, C25.1, C29.+, R12.1, R13.1, SV1.3, SV2.3, U$1.VDD, U$1.VDD@2, U$1.VDD@3, U$1.VDDA, U$1.VDDIO2, U$11.VIN, U$14.DIR, U$14.VCCA, U$15.VCC+, U$16.VCC, U$2.+VS, U$4.VD, U$6.VOUT
- net GND: now also C10.2, C11.2, C12.2, C13.2, C14.2, C16.2, C17.2, C18.1, C18.2, C20.2, C21.2, C22.2, C23.2, C24.2, C25.2, C26.-, C27.-, C28.-, C29.-, C3.2, C30.-, C4.2, C7.2, C8.2, C9.2, D1.A, K11.2, LED1.C, R4.1, R7.2, S1.P, S1.P1, S2.P, S2.P1, SV1.4, SV2.4, U$1.VSS, U$1.VSS@2, U$1.VSS@3, U$1.VSSA, U$10.P$2, U$11.GND, U$12.P$2, U$13.GND, U$14.GND, U$15.VCC-, U$16.GND, U$2.-VS, U$2.REF, U$3.-VDC, U$6.GND, U$7.V-
- net N$1: now also U$3.VAC-L
- net N$2: now also F1.1, U$5.P$2
- net N$3: now also U$5.P$1, U$8.P$2
- net N$4: now also U$8.P$1
Other:
- note added: "AC/DC Conversion"
- note added: "Debuging Interface"
- note added: "Flow Sensor"
- note added: "PA10 -> USART1_RX PA9 -> USART1_TX"
- note added: "PC4 -> USART3_RX PC5 -> USART3_TX"
- note added: "Programming Interface"
- note added: "Pump Power"
- note added: "Thermocouple Amplifier"
- note added: "~100nF"
- moved on the sheet: C1, C10, C2, C3, C4, C5, C6, C7, C8, C9, K1, SV1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

Commit message: Finished schematic and board files
Parts:
- removed C10, C25, C8: 4.7u, rcl:C-USC0805
- removed C11: 1u, rcl:C-USC0805
- removed C12, C19: 10n, rcl:C-USC0805
- removed C2, C22, C23, C24, C3, C4, C5, C6, C7, C9: 100n, rcl:C-USC0805
- removed C26, C27, C28, C29, C30: 470u, rcl:CPOL-USUD-10X10
- removed D1: BAS70, diode:BAS70
- removed F1: FUSEBLANK_5X20MM, fuse:FUSEBLANK_5X20MM
- removed R3: 27k, rcl:R-US_R0805
- removed R4: 10k, rcl:R-US_R0805
- removed S1, S2: (no value), switch-omron:10-XX
- removed SV1: (no value), con-lstb:MA04-1
- removed U$10, U$8, U$9: 5TERM, EmbSystems:5TERM
- removed U$12: 5TERM-3, EmbSystems:5TERM-3
- removed U$13: LD117-5, EmbSystems:LD117-5
- removed U$14: 74LVC, EmbSystems:74LVC
- removed U$15: LMV321LICT, EmbSystems:LMV321LICT
- removed U$16: NC7SZ04, EmbSystems:NC7SZ04
- added SV3, SV4: (no value), con-lstb:MA03-1
- C1: value 4.7u -> 10n
- R1: value P593 -> 10k; device varistor:P593 -> rcl:R-US_R0805
- SV2: device con-lstb:MA04-1 -> con-lstb:MA08-1
- U$1: value STM32F072RBT6 -> 5TERM; device EmbSystems:STM32F072RBT6 -> EmbSystems:5TERM
- U$3: value RAC20-N -> 5TERM; device EmbSystems:RAC20-N -> EmbSystems:5TERM
- U$6: value LD1117-3V3 -> 5TERM; device EmbSystems:LD1117-3V3 -> EmbSystems:5TERM
- U$7: value LT1206 -> 5TERM; device EmbSystems:LT1206 -> EmbSystems:5TERM
Connections:
- removed net 12V: C26.+, C27.+, C28.+, U$13.VIN, U$3.+VDC, U$6.VIN, U$7.V+
- removed net BREW: S2.S, S2.S1, U$1.PA6
- removed net DAC_OUT1: U$1.PA4, U$7.+IN
- removed net N$10: C19.2, U$7.COMP
- removed net N$11: C19.1, D1.C, R3.2, U$10.P$1, U$7.OUT
- removed net N$12: R3.1, R4.2, U$7.-IN
- removed net N$15: U$15.IN-, U$15.OUT, U$7.S/D
- removed net N$17: U$12.P$1, U$14.B
- removed net NRST: U$1.NRST, U$16.OUT
- removed net PA10: SV2.2, U$1.PA10
- removed net PA9: SV2.1, U$1.PA9
- removed net PC4: SV1.2, U$1.PC4
- removed net PC5: SV1.1, U$1.PC5
- removed net PUMPSHUTDOWN: U$1.PB15, U$15.IN+
- removed net RST: S1.S, S1.S1
- net 3V3: now also SV2.1; no longer C1.1, C10.1, C11.1, C12.1, C2.1, C22.1, C23.1, C24.1, C25.1, C29.+, C3.1, C4.1, C5.1, C6.1, C7.1, C8.1, C9.1, SV1.3, SV2.3, U$1.VDD, U$1.VDD@2, U$1.VDD@3, U$1.VDDA, U$1.VDDIO2, U$14.DIR, U$14.VCCA, U$15.VCC+, U$16.VCC, U$6.VOUT
- net 5V: now also SV2.3, U$6.P$1; no longer C30.+, U$12.P$3, U$13.VOUT, U$14.VCCB
- net ADC_IN1: now also SV3.2; no longer U$1.PA1
- net ENCA: now also SV2.6; no longer U$1.PA2
- net ENCB: now also SV2.7; no longer U$1.PA3
- net FLOW: now also C1.1, R1.2, SV2.5; no longer U$1.PA5, U$14.A
- net GND: now also SV2.2, SV3.1, SV3.3, U$6.P$2, U$7.P$2; no longer C10.2, C11.2, C12.2, C2.2, C22.2, C23.2, C24.2, C25.2, C26.-, C27.-, C28.-, C29.-, C3.2, C30.-, C4.2, C5.2, C6.2, C7.2, C8.2, C9.2, D1.A, R4.1, S1.P, S1.P1, S2.P, S2.P1, SV1.4, SV2.4, U$1.VSS, U$1.VSS@2, U$1.VSS@3, U$1.VSS@4, U$1.VSSA, U$10.P$2, U$12.P$2, U$13.GND, U$14.GND, U$15.VCC-, U$16.GND, U$3.-VDC, U$6.GND, U$7.V-
- net I2C1_SCL: now also SV4.2; no longer U$1.PB6
- net I2C1_SDA: now also SV4.1; no longer U$1.PB7
- net N$1: now also R1.1, U$7.P$1; no longer F1.2, U$3.VAC-L
- net N$2: no longer F1.1, R1.2
- net N$3: now also U$3.P$2; no longer R1.1, U$3.VAC-R, U$8.P$2
- net N$4: now also U$3.P$1; no longer U$8.P$1
- net N$8: now also U$1.P$2; no longer U$9.P$2
- net N$9: now also U$1.P$1; no longer U$9.P$1
- net RELAY: now also SV2.8; no longer U$1.PB12
- net SRST: now also SV4.3; no longer U$1.PB5
- net SW: now also SV2.4; no longer U$1.PA0
Other:
- note removed: "AC/DC Conversion"
- note removed: "Debuging Interface"
- note removed: "PA10 -> USART1_RX PA9 -> USART1_TX"
- note removed: "PC4 -> USART3_RX PC5 -> USART3_TX"
- note removed: "Programming Interface"
- note removed: "Pump Power"
- moved on the sheet: C1, C13, C14, C15, C16, C17, C18, C20, C21, K1, LED1, R10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
